Commit message: fix: add finger mass to fix gazebo model shake

File: ABBRobots/IRB120/irb120_ros2_gazebo/urdf/irb120_macro.urdf.xacro (robot description, xacro)
@@ -317,5 +317,5 @@
         <inertial>
           <origin xyz="0 0 0" rpy="0 0 ${pi/4}" />
-          <mass value="0.001" />
+          <mass value="0.2" />
           <inertia ixx="0.001" ixy="0.0" ixz="0.0" iyy="0.001" iyz="0.0" izz="0.001"/>
         </inertial>
@@ -335,5 +335,5 @@
         <inertial>
           <origin xyz="0 0 0" rpy="0 0 0" />
-          <mass value="0.005" />
+          <mass value="1.0" />
           <inertia ixx="0.001" ixy="0.0" ixz="0.0" iyy="0.001" iyz="0.0" izz="0.001"/>
         </inertial>
@@ -362,5 +362,5 @@
         <inertial>
           <origin xyz="0.01483 -0.00782 0" rpy="0 0 0" />
-          <mass value="0.002" />
+          <mass value="0.2" />
           <inertia ixx="0.001" ixy="0.0" ixz="0.0" iyy="0.001" iyz="0.0" izz="0.001"/>
         </inertial>
@@ -383,5 +383,5 @@
         <parent link="egp64_gripper_base_link" />
         <child link="egp64_finger_left_link" />
-        <limit effort="100" lower="-0.001" upper="0.04" velocity="0.2"/>
+        <limit effort="100" lower="-0.01" upper="0.025" velocity="0.2"/>
         <origin xyz="0.01483 -0.00782 0" rpy="0 0 0" />
         <axis xyz="-1 0 0" />
@@ -392,5 +392,5 @@
         <inertial>
           <origin xyz="0.03869 -0.0005 0.00093" rpy="0 0 0" />
-          <mass value="0.001" />
+          <mass value="0.1" />
           <inertia ixx="0.001" ixy="0.0" ixz="0.0" iyy="0.001" iyz="0.0" izz="0.001"/>
         </inertial>
@@ -419,5 +419,5 @@
         <inertial>
           <origin xyz="-0.0153 -0.00602 0" rpy="0 0 0" />
-          <mass value="0.002" />
+          <mass value="0.2" />
           <inertia ixx="0.001" ixy="0.0" ixz="0.0" iyy="0.001" iyz="0.0" izz="0.001"/>
         </inertial>
@@ -438,14 +438,13 @@
         <parent link="egp64_gripper_base_link" />
         <child link="egp64_finger_right_link" />
-        <limit effort="100" lower="-0.001" upper="0.04" velocity="0.2"/>
+        <limit effort="100" lower="-0.01" upper="0.025" velocity="0.2"/>
         <origin xyz="-0.0153 -0.00602 0" rpy="0 0 0" />
         <axis xyz="1 0 0" />
         <dynamics damping="1.0" friction="1.0"/>
       </joint>
-      <!-- RIGHT FINGERTIP -->
       <link name="egp64_fingertip_right_link">
         <inertial>
           <origin xyz="-0.01211 -0.00197 0.00093" rpy="0 0 0" />
-          <mass value="0.001" />
+          <mass value="0.1" />
           <inertia ixx="0.001" ixy="0.0" ixz="0.0" iyy="0.001" iyz="0.0" izz="0.001"/>
         </inertial>
@@ -472,5 +471,5 @@
         <inertial>
           <origin xyz="0 0 0" rpy="0 0 0" />
-          <mass value="0.00001" />
+          <mass value="0.1" />
           <inertia ixx="0.001" ixy="0.0" ixz="0.0" iyy="0.001" iyz="0.0" izz="0.001"/>
         </inertial>

Commit message: perf: Set the gripper finger straight

File: ABBRobots/IRB120/irb120_ros2_gazebo/urdf/irb120_macro.urdf.xacro (robot description, xacro)
@@ -323,5 +323,6 @@
       <!-- Schunk coupler (JOINT): -->
       <joint name="schunk_coupler_joint" type="fixed">
-        <origin xyz="0 0 0.001" rpy="0 0 ${pi/4}" />
+        <!-- <origin xyz="0 0 0.001" rpy="0 0 ${pi/4}" /> -->
+        <origin xyz="0 0 0.001" rpy="0 0 ${pi/2}" />
         <parent link="tool0"/>
         <child link="schunk_coupler"/>

Commit message: perf: Confirm TCP is [0,0,0.2]

File: ABBRobots/IRB120/irb120_ros2_gazebo/urdf/irb120_macro.urdf.xacro (robot description, xacro)
@@ -357,5 +357,5 @@
         <parent link="schunk_coupler"/>
         <child link="egp64_gripper_base_link"/>
-        <origin xyz="-0.03205 0.01812 0.02047" rpy="0 0 0" />
+        <origin xyz="-0.03205 0.01812 0.02" rpy="0 0 0" />
       </joint>
       <!-- LEFT FINGER BASE -->
@@ -486,5 +486,5 @@
         <limit effort="10000" lower="0.0" upper="0.0" velocity="0.0"/>
         <axis xyz="1 0 0" />
-        <origin xyz="0.033 -0.018 0.15" rpy="0 0 0"/>
+        <origin xyz="0.033 -0.018 0.179" rpy="0 0 0"/>
         <dynamics damping="1.0" friction="1.0"/>
       </joint>

Commit message: perf: Add EE_egp64v visual mesh for calibration

File: ABBRobots/IRB120/irb120_ros2_gazebo/urdf/irb120_macro.urdf.xacro (robot description, xacro)
@@ -478,4 +478,5 @@
           <geometry>
             <box size= "0.001 0.001 0.001" />
+            <!-- <mesh filename="file://$(find irb120_ros2_gazebo)/meshes/cube/meshes/model.dae" /> -->
           </geometry>
         </visual>

Commit message: perf: Finish pick and place simulation

File: ABBRobots/IRB120/irb120_ros2_gazebo/urdf/irb120_macro.urdf.xacro (robot description, xacro)
@@ -384,5 +384,5 @@
         <parent link="egp64_gripper_base_link" />
         <child link="egp64_finger_left_link" />
-        <limit effort="100" lower="-0.01" upper="0.025" velocity="0.2"/>
+        <limit effort="100" lower="-0.02" upper="0.025" velocity="0.2"/>
         <origin xyz="0.01483 -0.00782 0" rpy="0 0 0" />
         <axis xyz="-1 0 0" />
@@ -439,5 +439,5 @@
         <parent link="egp64_gripper_base_link" />
         <child link="egp64_finger_right_link" />
-        <limit effort="100" lower="-0.01" upper="0.025" velocity="0.2"/>
+        <limit effort="100" lower="-0.02" upper="0.025" velocity="0.2"/>
         <origin xyz="-0.0153 -0.00602 0" rpy="0 0 0" />
         <axis xyz="1 0 0" />

Commit message: perf: Add hollow cube generate xacro file

File: ABBRobots/IRB120/irb120_ros2_gazebo/urdf/irb120_macro.urdf.xacro (robot description, xacro)
@@ -384,5 +384,5 @@
         <parent link="egp64_gripper_base_link" />
         <child link="egp64_finger_left_link" />
-        <limit effort="100" lower="-0.02" upper="0.025" velocity="0.2"/>
+        <limit effort="100" lower="-0.00" upper="0.025" velocity="0.2"/>
         <origin xyz="0.01483 -0.00782 0" rpy="0 0 0" />
         <axis xyz="-1 0 0" />
@@ -439,5 +439,5 @@
         <parent link="egp64_gripper_base_link" />
         <child link="egp64_finger_right_link" />
-        <limit effort="100" lower="-0.02" upper="0.025" velocity="0.2"/>
+        <limit effort="100" lower="-0.0" upper="0.025" velocity="0.2"/>
         <origin xyz="-0.0153 -0.00602 0" rpy="0 0 0" />
         <axis xyz="1 0 0" />
