Commit message: perf: Add RGBD_Camera

File: ABBRobots/IRB120/irb120_ros2_gazebo/urdf/irb120.urdf.xacro (robot description, xacro)
@@ -48,4 +48,56 @@
 -->
 <robot name="irb120" xmlns:xacro="http://ros.org/wiki/xacro">
+  <link name="camera_link">
+    <collision name="camera_link_collision">
+      <geometry>
+        <box size="0.1 0.1 0.05"/>
+      </geometry>
+      <origin rpy="0 0 0" xyz="0 0 0"/>
+    </collision>
+    <visual name="camera_link_visual">
+      <geometry>
+        <box size="0.1 0.1 0.05"/>
+      </geometry>
+      <origin rpy="0 0 0" xyz="0 0 0"/>
+    </visual>
+    <inertial>
+      <mass value="2"/>
+      <inertia ixx="0.1" ixy="0.0" ixz="0.0" iyy="0.1" iyz="0.0" izz="0.1"/>
+    </inertial>
+  </link>
+  <joint name="camera_joint" type="fixed">
+    <parent link="base_link"/>
+    <child link = "camera_link"/>
+    <origin xyz="0.35 -0.3 1.0" rpy="0.0 ${pi} ${pi/2}"/>
+  </joint>
+  <gazebo reference="base_link">
+    <sensor name="RGBD_camera" type="depth">
+      <always_on>true</always_on>
+      <update_rate>1</update_rate>
+      <!-- Default pose wrt to world is [0 0 0 -pi/2 0 -pi/2] (xyz, rpy) -->
+      <!-- camera Z = world X, camera Y = world -Z, camera X = world -Y -->
+      <!-- x y z R P Y -->
+      <pose>0.35 -0.3 1.0 0.0 ${pi/2} 0.0</pose>
+      <camera name="realsense_depth_camera">
+        <horizontal_fov>0.6</horizontal_fov>
+        <image>
+          <width>320</width>
+          <height>240</height>
+          <format>B8G8R8</format>
+        </image>
+        <clip>
+          <near>0.5</near>
+          <far>1.5</far>
+        </clip>
+      </camera>
+      <plugin name="camera_controller" filename="libgazebo_ros_camera.so">
+        <camera_name>RGBD_camera</camera_name>
+        <frame_name>camera_link</frame_name>
+        <hack_baseline>0.07</hack_baseline>
+        <min_depth>0.05</min_depth>
+        <max_depth>8.0</max_depth>
+      </plugin>
+    </sensor>
+  </gazebo>
   <!-- ===== ARGUMENTS ===== -->
   <!-- CELL LAYOUT:  -->

File: ABBRobots/IRB120/irb120_ros2_gazebo/urdf/irb120_macro.urdf.xacro (robot description, xacro)
@@ -386,5 +386,5 @@
         <origin xyz="0.01483 -0.00782 0" rpy="0 0 0" />
         <axis xyz="-1 0 0" />
-        <dynamics damping="1.0" friction="1.0"/>
+        <dynamics damping="10.0" friction="0.1"/>
       </joint>
       <!-- LEFT FINGERTIP -->
@@ -441,5 +441,5 @@
         <origin xyz="-0.0153 -0.00602 0" rpy="0 0 0" />
         <axis xyz="1 0 0" />
-        <dynamics damping="1.0" friction="1.0"/>
+        <dynamics damping="10.0" friction="0.1"/>
       </joint>
       <link name="egp64_fingertip_right_link">

Commit message: perf: Add gazebo grasp fix package and could grasp

File: ABBRobots/IRB120/irb120_ros2_gazebo/urdf/irb120.urdf.xacro (robot description, xacro)
@@ -100,4 +100,26 @@
     </sensor>
   </gazebo>
+  <gazebo>
+      <plugin name="gazebo_grasp_fix" filename="libgazebo_grasp_fix.so">
+        <!--
+              NOTE: The finger tips are linked together with the links before, because they are connected with a
+        fixed joint. Gazebo makes one whole link out of this automatically. When listing the 9_*_tip links
+        here, they won't be found in the SDF.
+              -->
+              <arm>
+                  <arm_name>irb120</arm_name>
+                  <palm_link>EE_egp64</palm_link>
+                  <gripper_link>egp64_finger_left_link</gripper_link>
+                  <gripper_link>egp64_finger_right_link</gripper_link>
+              </arm>
+        <forces_angle_tolerance>100</forces_angle_tolerance>
+        <update_rate>30</update_rate>
+        <grip_count_threshold>4</grip_count_threshold>
+        <max_grip_count>8</max_grip_count>
+        <release_tolerance>0.005</release_tolerance>
+        <disable_collisions_on_attach>false</disable_collisions_on_attach>
+        <contact_topic>__default_topic__</contact_topic>
+      </plugin>
+    </gazebo>
   <!-- ===== ARGUMENTS ===== -->
   <!-- CELL LAYOUT:  -->

File: ABBRobots/IRB120/irb120_ros2_gazebo/urdf/irb120_ros2control.xacro (robot description, xacro)
@@ -165,12 +165,4 @@
         <!-- egp64_finger_left_joint -->
         <joint name="egp64_finger_left_joint">
-          <command_interface name="position">
-            <param name="min">-0.001</param>
-            <param name="max">0.04</param>
-          </command_interface>
-          <command_interface name="velocity">
-            <param name="min">-0.2</param>
-            <param name="max">0.2</param>
-          </command_interface>
           <command_interface name="effort">
             <param name="min">-100</param>
@@ -183,12 +175,4 @@
         <!-- egp64_finger_right_joint -->
         <joint name="egp64_finger_right_joint">
-          <command_interface name="position">
-            <param name="min">-0.001</param>
-            <param name="max">0.04</param>
-          </command_interface>
-          <command_interface name="velocity">
-            <param name="min">-0.2</param>
-            <param name="max">0.2</param>
-          </command_interface>
           <command_interface name="effort">
             <param name="min">-100</param>
@@ -243,16 +227,30 @@
       <gazebo reference="egp64_gripper_base_link">
         <selfCollide>false</selfCollide>
+        <mu1>1.0</mu1>
+        <mu2>1.0</mu2>
       </gazebo>
       <gazebo reference="egp64_finger_left_link">
         <selfCollide>false</selfCollide>
+        <mu1>1.0</mu1>
+        <mu2>1.0</mu2>
+        <material>Gazebo/Black</material>
       </gazebo>
       <gazebo reference="egp64_fingertip_left_link">
         <selfCollide>false</selfCollide>
+        <mu1>1.0</mu1>
+        <mu2>1.0</mu2>
+        <material>Gazebo/Black</material>
       </gazebo>
       <gazebo reference="egp64_finger_right_link">
         <selfCollide>false</selfCollide>
+        <mu1>1.0</mu1>
+        <mu2>1.0</mu2>
+        <material>Gazebo/Black</material>
       </gazebo>
       <gazebo reference="egp64_fingertip_right_link">
         <selfCollide>false</selfCollide>
+        <mu1>1.0</mu1>
+        <mu2>1.0</mu2>
+        <material>Gazebo/Black</material>
       </gazebo>
     </xacro:if>

Commit message: perf: Add camera and model dae with texture

File: ABBRobots/IRB120/irb120_ros2_gazebo/urdf/irb120.urdf.xacro (robot description, xacro)
@@ -56,8 +56,8 @@
     </collision>
     <visual name="camera_link_visual">
+      <origin xyz="0 0 0" rpy="0 0 0"/>
       <geometry>
-        <box size="0.1 0.1 0.05"/>
+        <mesh filename="file://$(find irb120_ros2_gazebo)/meshes/camera/EpicEyeS-M.dae"/>
       </geometry>
-      <origin rpy="0 0 0" xyz="0 0 0"/>
     </visual>
     <inertial>

File: ABBRobots/IRB120/irb120_ros2_gazebo/urdf/irb120_ros2control.xacro (robot description, xacro)
@@ -229,4 +229,5 @@
         <mu1>1.0</mu1>
         <mu2>1.0</mu2>
+        <material>Gazebo/Grey</material>
       </gazebo>
       <gazebo reference="egp64_finger_left_link">
@@ -240,17 +241,17 @@
         <mu1>1.0</mu1>
         <mu2>1.0</mu2>
+        <material>Gazebo/White</material>
+      </gazebo>
+      <gazebo reference="egp64_finger_right_link">
+        <selfCollide>false</selfCollide>
+        <mu1>1.0</mu1>
+        <mu2>1.0</mu2>
         <material>Gazebo/Black</material>
       </gazebo>
-      <gazebo reference="egp64_finger_right_link">
-        <selfCollide>false</selfCollide>
-        <mu1>1.0</mu1>
-        <mu2>1.0</mu2>
-        <material>Gazebo/Black</material>
-      </gazebo>
       <gazebo reference="egp64_fingertip_right_link">
         <selfCollide>false</selfCollide>
         <mu1>1.0</mu1>
         <mu2>1.0</mu2>
-        <material>Gazebo/Black</material>
+        <material>Gazebo/White</material>
       </gazebo>
     </xacro:if>

Commit message: perf: Add 2D camera for print screen

File: ABBRobots/IRB120/irb120_ros2_gazebo/urdf/irb120.urdf.xacro (robot description, xacro)
@@ -100,4 +100,63 @@
     </sensor>
   </gazebo>
+  <link name="camera_link_2D">
+    <collision name="camera_link_collision">
+      <geometry>
+        <box size="0.02 0.02 0.04"/>
+      </geometry>
+      <origin rpy="0 0 0" xyz="0 0 0"/>
+    </collision>
+    <visual name="camera_link_visual">
+      <geometry>
+        <box size="0.01 0.02 0.03"/>
+      </geometry>
+      <origin rpy="0 0 0" xyz="0 0 0"/>
+    </visual>
+  </link>
+  <joint name="camera_joint_2D" type="fixed">
+    <parent link="base_link"/>
+    <child link = "camera_link_2D"/>
+    <origin xyz="0.0 0.573971 0.7" rpy="0.0 ${pi/2} 0.0"/>
+  </joint>
+  <!-- camera -->
+  <gazebo reference="camera_link_2D">
+    <sensor type="camera" name="camera1">
+      <update_rate>1.0</update_rate>
+      <camera name="head">
+        <horizontal_fov>1.3962634</horizontal_fov>
+        <image>
+          <width>2000</width>
+          <height>2000</height>
+          <format>R8G8B8</format>
+        </image>
+        <clip>
+          <near>0.02</near>
+          <far>300</far>
+        </clip>
+        <noise>
+          <type>gaussian</type>
+          <!-- Noise is sampled independently per pixel on each frame.
+               That pixel's noise value is added to each of its color
+               channels, which at that point lie in the range [0,1]. -->
+          <mean>0.0</mean>
+          <stddev>0.0</stddev>
+        </noise>
+      </camera>
+      <plugin name="camera_controller_2D" filename="libgazebo_ros_camera.so">
+        <alwaysOn>true</alwaysOn>
+        <updateRate>0.0</updateRate>
+        <cameraName>camera_2D</cameraName>
+        <imageTopicName>image_raw</imageTopicName>
+        <cameraInfoTopicName>camera_info</cameraInfoTopicName>
+        <frameName>camera_link_2D</frameName>
+        <hackBaseline>0.07</hackBaseline>
+        <distortionK1>0.0</distortionK1>
+        <distortionK2>0.0</distortionK2>
+        <distortionK3>0.0</distortionK3>
+        <distortionT1>0.0</distortionT1>
+        <distortionT2>0.0</distortionT2>
+      </plugin>
+    </sensor>
+  </gazebo>
   <gazebo>
       <plugin name="gazebo_grasp_fix" filename="libgazebo_grasp_fix.so">

Commit message: perf: Add grasp fix update rate and add gripper range

File: ABBRobots/IRB120/irb120_ros2_gazebo/urdf/irb120.urdf.xacro (robot description, xacro)
@@ -177,5 +177,5 @@
               </arm>
         <forces_angle_tolerance>100</forces_angle_tolerance>
-        <update_rate>30</update_rate>
+        <update_rate>60</update_rate>
         <grip_count_threshold>4</grip_count_threshold>
         <max_grip_count>8</max_grip_count>

File: ABBRobots/IRB120/irb120_ros2_gazebo/urdf/irb120_macro.urdf.xacro (robot description, xacro)
@@ -273,5 +273,6 @@
       <parent link="${prefix}link_5"/>
       <child link="${prefix}link_6"/>
-      <limit effort="0" lower="-6.98132" upper="6.98132" velocity="7.33038"/>
+      <!-- <limit effort="0" lower="-6.98132" upper="6.98132" velocity="7.33038"/> -->
+      <limit effort="0" lower="-3.1415926" upper="3.1415926" velocity="7.33038"/>
       <axis xyz="1 0 0"/>
       <dynamics damping="1.0" friction="1.0"/>
@@ -384,5 +385,5 @@
         <parent link="egp64_gripper_base_link" />
         <child link="egp64_finger_left_link" />
-        <limit effort="100" lower="-0.00" upper="0.025" velocity="0.2"/>
+        <limit effort="100" lower="-0.02" upper="0.025" velocity="0.2"/>
         <origin xyz="0.01483 -0.00782 0" rpy="0 0 0" />
         <axis xyz="-1 0 0" />
@@ -439,5 +440,5 @@
         <parent link="egp64_gripper_base_link" />
         <child link="egp64_finger_right_link" />
-        <limit effort="100" lower="-0.0" upper="0.025" velocity="0.2"/>
+        <limit effort="100" lower="-0.02" upper="0.025" velocity="0.2"/>
         <origin xyz="-0.0153 -0.00602 0" rpy="0 0 0" />
         <axis xyz="1 0 0" />
